File: ledusbc2key/ledusbc2key.sch (KiCad schematic (older format))
At the start: 18 parts

Commit message: starting pcb file
Parts:
- added D1, D2: D_Small, Diode_SMD:D_SOD-123, symbol Device:D_Small
- added MX1, MX2: MX-NoLED, MX_Alps_Hybrid:MX-1U-NoLED, symbol MX_Alps_Hybrid:MX-NoLED
- added R5, R6: 5.1k, Resistor_SMD:R_0805_2012Metric_Pad1.15x1.40mm_HandSolder, symbol Device:R_Small
- added U2: PRTR5V0U2X, random-keyboard-parts:SOT143B, symbol random-keyboard-parts:PRTR5V0U2X
- C1, C2, C3, C4, C5, C6, C7, C8: renamed from C?; footprint (none) -> Capacitor_SMD:C_0805_2012Metric_Pad1.15x1.40mm_HandSolder
- F1: renamed from F?; footprint (none) -> Fuse:Fuse_1206_3216Metric_Pad1.42x1.75mm_HandSolder
- J1: renamed from J?; footprint (none) -> random-keyboard-parts:Reset_Pretty-Mask
- R1, R2, R3, R4: renamed from R?; footprint (none) -> Resistor_SMD:R_0805_2012Metric_Pad1.15x1.40mm_HandSolder
- SW1: renamed from SW?; footprint (none) -> random-keyboard-parts:PushButton_6x6mm_TH
- USB1: renamed from USB?; footprint (none) -> Type-C:HRO-TYPE-C-31-M-12-HandSoldering
- Y1: renamed from Y?; footprint (none) -> Crystal:Crystal_SMD_3225-4Pin_3.2x2.5mm_HandSoldering
- gave numbers to parts that had none: 1
Connections:
- net GND: now also USB1.1 (GND), USB1.12 (GND), USB1.13 (SHIELD), R5.2, R6.2, U2.1 (GND)
- net ROW0: now reaches U1.19 (PD1)
- net ROW0: now also D1.1 (K), D2.1 (K)
- net COL0: now reaches U1.20 (PD2)
- net COL0: now also MX1.1 (COL)
- net COL1: now reaches U1.21 (PD3)
- net COL1: now also MX2.1 (COL)
- net at USB1.10 (CC2): now also R5.1
- net at USB1.4 (CC1): now also R6.1
- net at R3.2, USB1.5 (DN2), USB1.7 (DN1): now also U2.3 (IO2)
- net at R4.2, USB1.6 (DP1), USB1.8 (DP2): now also U2.2 (IO1)
- new net: D1.2 (A), MX1.2 (ROW)
- new net: D2.2 (A), MX2.2 (ROW)
Other:
- moved on the sheet: R3, R4
